Commit message: [MOD-HW] Add Multi Motor Xacro and tests

File: mirte_modular_hardware/urdf/encoder.ros2_control.xacro (robot description, xacro)
@@ -1,4 +1,5 @@
 <?xml version="1.0"?>
 <robot xmlns:xacro="http://www.ros.org/wiki/xacro">
+  <xacro:include filename="$(find mirte_modular_hardware)/urdf/common.xacro" />
   <!-- NOTE; The standard slot encoders compatible with the yellow TT motors of the MIRTE Pioneer,
              have 20 ticks per rotations -->
@@ -6,7 +7,5 @@
     params="hardware_namespace:='io' hw_device_name joint_name ticks_per_rotation:=20 initial_message_timeout:=500">
     <!-- Strip leading slash -->
-    <xacro:property name="hardware_namespace_"
-      value="${hardware_namespace[:-1] if hardware_namespace[-1] == '/' else hardware_namespace}"
-      scope="parent" />
+    <xacro:strip_trailing_slash source="${hardware_namespace}" dest="hardware_namespace_" />
     <!-- <xacro:property name="topic_" value= scope="parent"/> -->
     <ros2_control name="mirte_modular_hardware_encoder_${hw_device_name}" type="sensor">

File: mirte_modular_hardware/urdf/motor.ros2_control.xacro (robot description, xacro)
@@ -1,10 +1,9 @@
 <?xml version="1.0"?>
 <robot xmlns:xacro="http://www.ros.org/wiki/xacro">
+  <xacro:include filename="$(find mirte_modular_hardware)/urdf/common.xacro" />
   <xacro:macro name="mirte_modular_hardware_motor"
     params="hardware_namespace:='io' hw_device_name joint_name max_motor_speed:='${6.0*pi}'">
-    <!-- Strip leading slash -->
-    <xacro:property name="hardware_namespace_"
-      value="${hardware_namespace[:-1] if hardware_namespace[-1] == '/' else hardware_namespace}"
-      scope="parent" />
+    <!-- Strip trailing slash -->
+    <xacro:strip_trailing_slash source="${hardware_namespace}" dest="hardware_namespace_" />
     <!-- <xacro:property name="topic_" value= scope="parent"/> -->
     <!-- NOTE; this *highly* depends on the voltage of the motors!!!! -->
