Commit message: Initial work in new mirte_master_control

File: mirte_modular_hardware/urdf/ros2_control.xacro (robot description, xacro)
@@ -1,10 +1,4 @@
 <?xml version="1.0"?>
 <robot xmlns:xacro="http://www.ros.org/wiki/xacro">
-  <!-- <xacro:macro name="command_interface" params="name min:='' max:=''"> -->
-  <!-- <xacro:if value="${any((min,max))}"> -->
-  <!-- ${xacro.error('not implemented')} -->
-  <!-- </xacro:if> -->
-  <!-- <command_interface name="${name}" /> -->
-  <!-- </xacro:macro> -->
   <xacro:macro name="optional_param" params="name value">
     <xacro:if value="${bool(value) or (python.isinstance(value, float|int) and bool(str(value)))}">
