Commit message: Remove package name prefix in favor of xacro namespacing
Namespace when necessary

File: mirte_control/mirte_pioneer_base_control/urdf/mirte_pioneer.ros2_control.xacro (robot description, xacro)
@@ -11,9 +11,9 @@
   <xacro:macro name="mirte_pioneer_base_control_motor"
     params="hardware_namespace:='io' hw_device_name joint_name ticks_per_rotation:=0 max_motor_speed='${6.0*pi}'">
-    <xacro:mirte_modular_hardware_motor hardware_namespace="${hardware_namespace}"
+    <xacro:motor_actuator hardware_namespace="${hardware_namespace}"
       hw_device_name="${hw_device_name}" joint_name="${joint_name}"
       max_motor_speed="${max_motor_speed}" />
     <xacro:if value="${ticks_per_rotation > 0}">
-      <xacro:mirte_modular_hardware_encoder hardware_namespace="${hardware_namespace}"
+      <xacro:encoder_sensor hardware_namespace="${hardware_namespace}"
         hw_device_name="${hw_device_name}" joint_name="${joint_name}"
         ticks_per_rotation="${ticks_per_rotation}" />

File: mirte_modular_hardware/test/encoder/test_encoder_basic.urdf.xacro (robot description, xacro)
@@ -28,4 +28,4 @@
     </visual>
   </link>
-  <xacro:mirte_modular_hardware_encoder hw_device_name="test_joint" joint_name="test_joint" />
+  <xacro:encoder_sensor hw_device_name="test_joint" joint_name="test_joint" />
 </robot>

File: mirte_modular_hardware/test/motor/test_motor_basic.urdf.xacro (robot description, xacro)
@@ -29,5 +29,5 @@
     </visual>
   </link>
-  <xacro:mirte_modular_hardware_encoder hw_device_name="test_encoder" joint_name="test_joint" />
-  <xacro:mirte_modular_hardware_motor hw_device_name="test_motor" joint_name="test_joint" />
+  <xacro:encoder_sensor hw_device_name="test_encoder" joint_name="test_joint" />
+  <xacro:motor_actuator hw_device_name="test_motor" joint_name="test_joint" />
 </robot>

File: mirte_modular_hardware/urdf/encoder.ros2_control.xacro (robot description, xacro)
@@ -4,5 +4,5 @@
   <!-- NOTE; The standard slot encoders compatible with the yellow TT motors of the MIRTE Pioneer,
              have 20 ticks per rotations -->
-  <xacro:macro name="mirte_modular_hardware_encoder"
+  <xacro:macro name="encoder_sensor"
     params="hardware_namespace:='io' hw_device_name joint_name ticks_per_rotation:=20 initial_message_timeout:=500">
     <!-- Strip leading slash -->

File: mirte_modular_hardware/urdf/motor.ros2_control.xacro (robot description, xacro)
@@ -2,5 +2,5 @@
 <robot xmlns:xacro="http://www.ros.org/wiki/xacro">
   <xacro:include filename="$(find mirte_modular_hardware)/urdf/common.xacro" />
-  <xacro:macro name="mirte_modular_hardware_motor"
+  <xacro:macro name="motor_actuator"
     params="hardware_namespace:='io' hw_device_name joint_name max_motor_speed:='${6.0*pi}'">
     <!-- Strip trailing slash -->
