Commit message: Rename package to mirte_master_control

File: mirte_control/mirte_master_control/urdf/mirte_master_base_multi_motor.ros2_control.xacro (robot description, xacro)
@@ -1,10 +1,10 @@
 <?xml version="1.0"?>
 <robot xmlns:xacro="http://www.ros.org/wiki/xacro">
-  <xacro:property name="config_file" value="$(find mirte_master_base_control)/config/default_hardware.yaml" />
+  <xacro:property name="config_file" value="$(find mirte_master_control)/config/default_hardware.yaml" />
   <xacro:property name="config" value="${xacro.load_yaml(config_file)}"/>
-  <xacro:include filename="$(find mirte_master_base_control)/urdf/multi_motor_actuator.ros2_control.xacro"/>
+  <xacro:include filename="$(find mirte_master_control)/urdf/multi_motor_actuator.ros2_control.xacro"/>
   <xacro:multi_motor_actuator base_config="${config.base}"/>
   <!-- For Now multi load encoders (could make merged encoder (1 hw multi sub) later) -->
-  <xacro:include filename="$(find mirte_master_base_control)/urdf/single_encoders.ros2_control.xacro" />
+  <xacro:include filename="$(find mirte_master_control)/urdf/single_encoders.ros2_control.xacro" />
   <xacro:single_encoders base_config="${config.base}"/>
 </robot>

File: mirte_control/mirte_master_control/urdf/mirte_master_base_single_motors.ros2_control.xacro (robot description, xacro)
@@ -1,11 +1,11 @@
 <?xml version="1.0"?>
 <robot xmlns:xacro="http://www.ros.org/wiki/xacro">
-  <xacro:property name="config_file" value="$(find mirte_master_base_control)/config/default_hardware.yaml" />
+  <xacro:property name="config_file" value="$(find mirte_master_control)/config/default_hardware.yaml" />
   <xacro:property name="config" value="${xacro.load_yaml(config_file)}"/>
   <!-- For Now multi load motors (could make merged motor (1 hw multi pub) later) -->
-  <xacro:include filename="$(find mirte_master_base_control)/urdf/single_motors.ros2_control.xacro" />
+  <xacro:include filename="$(find mirte_master_control)/urdf/single_motors.ros2_control.xacro" />
   <xacro:single_motors base_config="${config.base}"/>
   <!-- For Now multi load encoders (could make merged encoder (1 hw multi sub) later) -->
-  <xacro:include filename="$(find mirte_master_base_control)/urdf/single_encoders.ros2_control.xacro" />
+  <xacro:include filename="$(find mirte_master_control)/urdf/single_encoders.ros2_control.xacro" />
   <xacro:single_encoders base_config="${config.base}"/>
 </robot>

File: mirte_control/mirte_master_control/urdf/multi_motor_actuator.ros2_control.xacro (robot description, xacro)
@@ -3,5 +3,5 @@
   <xacro:macro name="multi_motor_actuator" params="base_config:=^|">
     <xacro:include filename="$(find mirte_modular_hardware)/urdf/multi_motor.ros2_control.xacro" />
-    <xacro:include filename="$(find mirte_master_base_control)/urdf/multi_motor_wheel_joints.xacro" />
+    <xacro:include filename="$(find mirte_master_control)/urdf/multi_motor_wheel_joints.xacro" />
     <xacro:property name="hardware_namespace" value="${base_config.hardware_namespace}" />
     <xacro:multi_motor_actuator hw_device_name="motorservocontroller" hardware_namespace="${hardware_namespace}">
