Commit message: Fix new control issues
Signed-off-by: SuperJappie08 <36795178+SuperJappie08@users.noreply.github.com>

File: mirte_control/mirte_master_control/urdf/base/motor/multi_motor.ros2_control.xacro (robot description, xacro)
@@ -10,15 +10,14 @@
       <!-- Wheel specific properties -->
       <xacro:property name="max_motor_speed" value="${wheel_config.max_motor_speed}" />
-      <xacro:property name="tmx_motor_name"
-        value="${wheel_config.get('tmx_motor_name', wheel_name)}" />
+      <xacro:property name="motor_name" value="${wheel_config.get('motor_name', wheel_name)}" />
       <xacro:property name="initial_value" value="${wheel_config.get('initial_motor_speed')}" />
       <!-- xacro:eval-comments:on -->
       <!-- wheel_name: ${wheel_name} -->
       <!-- max_motor_speed: ${max_motor_speed} -->
-      <!-- tmx_motor_name: ${tmx_motor_name} -->
+      <!-- motor_name: ${motor_name} -->
       <!-- initial_value(initial_motor_speed): ${initial_value} -->
       <!-- xacro:eval-comments:off -->
       <xacro:multi_motor_joint joint_name="${wheel_name}_wheel_joint"
-        max_motor_speed="${max_motor_speed}" tmx_motor_name="${tmx_motor_name}"
+        max_motor_speed="${max_motor_speed}" motor_name="${motor_name}"
         initial_value="${initial_value}" />
       <!-- recursively call myself -->

File: mirte_modular_hardware/test/multi_motor/multi_motor_simple.urdf.xacro (robot description, xacro)
@@ -54,5 +54,5 @@
       <xacro:multi_motor_joint
         joint_name="another_joint"
-        tmx_motor_name="top_left"
+        motor_name="top_left"
         max_motor_speed="10" />
     </joints>

File: mirte_modular_hardware/urdf/multi_motor.ros2_control.xacro (robot description, xacro)
@@ -17,7 +17,7 @@
   </xacro:macro>
   <xacro:macro name="multi_motor_joint"
-    params="joint_name tmx_motor_name:=${None} max_motor_speed initial_value:=${None}">
+    params="joint_name motor_name:=${None} max_motor_speed initial_value:=${None}">
     <joint name="${joint_name}">
-      <xacro:optional_param name="tmx_motor" value="${tmx_motor_name}" />
+      <xacro:optional_param name="motor_name" value="${motor_name}" />
       <command_interface name="velocity">
         <param name="max">${max_motor_speed}</param>
