Commit message: MIRTE Master description rework for control

File: mirte_control/mirte_master_control/urdf/base/encoder/single_encoders.ros2_control.xacro (robot description, xacro)
@@ -3,5 +3,5 @@
   <xacro:include filename="$(find mirte_modular_hardware)/urdf/encoder.ros2_control.xacro"/>
   <!-- Based on loop from xacro wiki -->
-  <xacro:macro name="single_encoders_loop" params="wheels:=^ base_config:=^">
+  <xacro:macro name="single_encoders_loop" params="wheels:=^ base_config:=^ hardware_namespace:=^|${None}">
       <xacro:if value="${wheels}">
       <!-- pop first item from list -->
@@ -9,5 +9,5 @@
       <xacro:property name="wheel_config" value="${base_config.wheels[wheel_name]}"/>
       <!-- Base properties -->
-      <xacro:property name="hardware_namespace" value="${base_config.get('hardware_namespace', 'io')}" />
+      <xacro:property name="hardware_namespace_" value="${hardware_namespace or base_config.get('hardware_namespace', 'io')}" />
       <xacro:property name="initial_message_timeout" value="${base_config.get('initial_message_timeout', 500)}" />
       <!-- Wheel specific properties -->
@@ -15,9 +15,9 @@
       <!-- xacro:eval-comments:on -->
       <!-- wheel_name: ${wheel_name} -->
-      <!-- hardware_namespace: ${hardware_namespace} -->
+      <!-- hardware_namespace: ${hardware_namespace_} -->
       <!-- initial_message_timeout: ${initial_message_timeout} ms -->
       <!-- ticks_per_rotation: ${ticks_per_rotation} -->
       <!-- xacro:eval-comments:off -->
-      <xacro:encoder_sensor hw_device_name="${wheel_name}" hardware_namespace="${hardware_namespace}"
+      <xacro:encoder_sensor hw_device_name="${wheel_name}" hardware_namespace="${hardware_namespace_}"
         joint_name="${wheel_name}_wheel_joint" initial_message_timeout="${initial_message_timeout}"
         ticks_per_rotation="${ticks_per_rotation}"
@@ -27,5 +27,5 @@
     </xacro:if>
   </xacro:macro>
-  <xacro:macro name="single_encoders" params="base_config:=^">
+  <xacro:macro name="encoders" params="base_config:=^ hardware_namespace:=^|${None}">
     <xacro:single_encoders_loop wheels="${list(base_config.wheels.keys())}" base_config="${base_config}" />
   </xacro:macro>

File: mirte_control/mirte_master_control/urdf/base/motor/single_motors.ros2_control.xacro (robot description, xacro)
@@ -3,5 +3,5 @@
   <xacro:include filename="$(find mirte_modular_hardware)/urdf/motor.ros2_control.xacro"/>
   <!-- Based on loop from xacro wiki -->
-  <xacro:macro name="single_motors_loop" params="wheels:=^ base_config:=^">
+  <xacro:macro name="single_motors_loop" params="wheels:=^ base_config:=^ hardware_namespace:=^|${None}">
       <xacro:if value="${wheels}">
       <!-- pop first item from list -->
@@ -9,13 +9,13 @@
       <xacro:property name="wheel_config" value="${base_config.wheels[wheel_name]}"/>
       <!-- Base properties -->
-      <xacro:property name="hardware_namespace" value="${base_config.get('hardware_namespace', 'io')}" />
+      <xacro:property name="hardware_namespace_" value="${hardware_namespace or base_config.get('hardware_namespace', 'io')}" />
       <!-- Wheel specific properties -->
       <xacro:property name="max_motor_speed" value="${wheel_config.max_motor_speed}"/>
       <!-- xacro:eval-comments:on -->
       <!-- wheel_name: ${wheel_name} -->
-      <!-- hardware_namespace: ${hardware_namespace} -->
+      <!-- hardware_namespace: ${hardware_namespace_} -->
       <!-- max_motor_speed: ${max_motor_speed} -->
       <!-- xacro:eval-comments:off -->
-      <xacro:motor_actuator hw_device_name="${wheel_name}" hardware_namespace="${hardware_namespace}"
+      <xacro:motor_actuator hw_device_name="${wheel_name}" hardware_namespace="${hardware_namespace_}"
         joint_name="${wheel_name}_wheel_joint" max_motor_speed="${max_motor_speed}" />
       <!-- recursively call myself -->
@@ -23,5 +23,5 @@
     </xacro:if>
   </xacro:macro>
-  <xacro:macro name="single_motors" params="base_config:=^">
+  <xacro:macro name="motors" params="base_config:=^ hardware_namespace:=^|${None}">
     <xacro:single_motors_loop wheels="${list(base_config.wheels.keys())}" base_config="${base_config}" />
   </xacro:macro>

File: mirte_control/mirte_pioneer_base_control/urdf/mirte_pioneer_combined.urdf.xacro (robot description, xacro)
@@ -6,9 +6,9 @@
   <!-- ticks per rotation, when set to 0, encoders are disabled. Default: 0 -->
   <xacro:arg name="ticks_per_rotation" default="0" />
-  <!-- NOTE; this *highly* depends on the voltage of the motors!!!! -->
+  <!-- NOTE: this *highly* depends on the voltage of the motors!!!! -->
   <!-- For 5V power bank; 255 pwm = 90 ticks/sec -> ca 2 rot/s (4*pi) -->
   <!-- For 6V power supply; 255 pwm = 120 ticks/sec -> ca 3 rot/s (6*pi) -->
   <xacro:arg name="max_motor_speed" default="${6.0*pi}" />
-  <!-- TODO(SuperJappie08) Add other param configurations  -->
+  <!-- TODO(SuperJappie08): Add other param configurations  -->
   <xacro:mirte_pioneer_base_control_motor hardware_namespace="$(arg hardware_namespace)"
     joint_name="joint_left_wheel" hw_device_name="left"

File: mirte_description/mirte_master_description/urdf/arm.xacro (robot description, xacro)
@@ -580,4 +580,5 @@
         <mimic joint="gripper_joint" multiplier="-1"/>
     </joint>
+<xacro:if value="$(arg include_old_sim_control)">
 <gazebo>
     <plugin filename="libgazebo_grasp_fix.so" name="gazebo_grasp_fix">
@@ -600,3 +601,4 @@
     </plugin>
 </gazebo>
+</xacro:if>
 </robot>

File: mirte_description/mirte_master_description/urdf/lidar.xacro (robot description, xacro)
@@ -72,5 +72,6 @@
     <xacro:property name="lidar_sensor_link" value="lidar_link" />
   </xacro:unless>
-  <gazebo reference="lidar_link">
+  <xacro:if value="$(arg include_old_sim_control)">
+    <gazebo reference="lidar_link">
         <sensor name="lidar" type="ray">
             <pose> 0 0 0 0 0 0 </pose>
@@ -101,3 +102,4 @@
         </sensor>
     </gazebo>
+  </xacro:if>
 </robot>

File: mirte_description/mirte_master_description/urdf/mirte_master.xacro (robot description, xacro)
@@ -2,4 +2,6 @@
 <robot
   name="mirte_master" xmlns:xacro="http://ros.org/wiki/xacro">
+  <!-- Whether to use include the old simulation and control setup or not -->
+  <xacro:arg name="include_old_sim_control" default="True" />
   <xacro:arg name="flag_enable" default="False" />
   <xacro:arg name="arm_enable" default="True" />
@@ -10,5 +12,7 @@
   <xacro:arg name="depth_camera_enable" default="True" />
   <xacro:arg name="imu_enable" default="True" />
-  <xacro:arg name="sim" default="False" />
+  <xacro:if value="$(arg include_old_sim_control)">
+    <xacro:arg name="sim" default="False" />
+  </xacro:if>
   <xacro:property name="camera_name" value="camera" lazy_eval="False"/>
   <xacro:property name="namespace" value="" scope="global" lazy_eval="False"/>
@@ -25,9 +29,11 @@
     <color rgba="0.203125 0.23828125 0.28515625 1.0" />
   </material>
-  <xacro:include filename="$(find mirte_master_description)/urdf/mirte_master_base.gazebo.xacro" />
+  <xacro:if value="$(arg include_old_sim_control)">
+    <xacro:include filename="$(find mirte_master_description)/urdf/mirte_master_base.gazebo.xacro" />
+  </xacro:if>
   <xacro:if value="$(arg depth_camera_enable)">
     <xacro:include filename="$(find mirte_master_description)/urdf/orbbec_astra_plus_pro.xacro" />
     <xacro:sensor_orbbec_astra_pro_plus name="${camera_name}" parent="frame_link" color="blue">
-      <origin xyz="0.01 -0.146658788505756 0.0427" rpy="0 0 ${radians(-90)}" />
+      <origin xyz="0.01 -0.146658788505756 0.0427" rpy="0 0 ${radians(-90)}" use_gazebo="$(arg include_old_sim_control)" />
     </xacro:sensor_orbbec_astra_pro_plus>
   </xacro:if>
@@ -41,7 +47,9 @@
   </xacro:if>
   <link name="base_link" />
-  <gazebo reference="base_link">
-     <kinematic>1</kinematic>
-  </gazebo>
+  <xacro:if value="$(arg include_old_sim_control)">
+    <gazebo reference="base_link">
+      <kinematic>1</kinematic>
+    </gazebo>
+  </xacro:if>
   <joint name="frame_base_joint" type="fixed">
     <origin xyz="0 0 0.10" rpy="0 0 ${radians(90)}" />
@@ -169,20 +177,20 @@
     </joint>
     <link name="link_chassis" />
-    <xacro:ultrasonic_sensor name="front_left">
+    <xacro:ultrasonic_sensor name="front_left" with_gazebo="$(arg include_old_sim_control)">
       <origin
         xyz="0.05297775289576 -0.120282421780502 -0.031"
         rpy="0 0 ${-pi/2+0.296705972839036}" />
     </xacro:ultrasonic_sensor>
-    <xacro:ultrasonic_sensor name="front_right">
+    <xacro:ultrasonic_sensor name="front_right" with_gazebo="$(arg include_old_sim_control)">
       <origin
         xyz="-0.05297775289576 -0.120282421780502 -0.031"
         rpy="0 0 ${-pi/2-0.296705972839036}" />
     </xacro:ultrasonic_sensor>
-    <xacro:ultrasonic_sensor name="rear_left">
+    <xacro:ultrasonic_sensor name="rear_left" with_gazebo="$(arg include_old_sim_control)">
       <origin
         xyz="0.0565606470918482 0.119187021096338 -0.031"
         rpy="0 0 ${-pi/2 + 2.84488668075076}" />
     </xacro:ultrasonic_sensor>
-    <xacro:ultrasonic_sensor name="rear_right">
+    <xacro:ultrasonic_sensor name="rear_right" with_gazebo="$(arg include_old_sim_control)">
       <origin
         xyz="-0.0565606470918482 0.119187021096338 -0.031"

File: mirte_description/mirte_master_description/urdf/orbbec_astra_plus_pro.xacro (robot description, xacro)
@@ -13,5 +13,5 @@
      <xacro:property name="M_PI" value="3.1415926535897931" />
      <xacro:macro name="sensor_orbbec_astra_pro_plus"
-          params="name parent *origin color rgb_w:=640 rgb_h:=480 stddev:=0.5">
+          params="name parent *origin color rgb_w:=640 rgb_h:=480 stddev:=0.5 with_gazebo:=True">
           <joint name="${name}_rgb_joint" type="fixed">
                <xacro:insert_block name="origin" />
@@ -93,6 +93,8 @@
                </inertial-->
           </link>
-          <!-- RGBD sensor for simulation, same as Kinect -->
-          <xacro:sensor_orbbec_astra_pro_plus_gazebo />
+          <xacro:if value="${with_gazebo}">
+               <!-- RGBD sensor for simulation, same as Kinect -->
+               <xacro:sensor_orbbec_astra_pro_plus_gazebo />
+          </xacro:if>
      </xacro:macro>
      <!-- ====================================================

File: mirte_description/mirte_master_description/urdf/ultrasonic.xacro (robot description, xacro)
@@ -3,5 +3,5 @@
 <!-- Modified to remove the collision and change the minimum distance -->
 <robot xmlns:xacro="http://www.ros.org/wiki/xacro">
-  <xacro:macro name="ultrasonic_sensor" params="name *origin">
+  <xacro:macro name="ultrasonic_sensor" params="name *origin with_gazebo:=True">
     <xacro:property name="sonar_angle_max" value="${radians(15)}"/>
     <joint name="sonar_${name}" type="fixed">
@@ -26,4 +26,5 @@
       </collision>
     </link>
+    <xacro:if value="${with_gazebo}">
     <gazebo reference="${name}_sonar">
       <sensor type="ray" name="range_sensor_${name}">
@@ -69,4 +70,5 @@
      </sensor>
    </gazebo>
+  </xacro:if>
   </xacro:macro>
 </robot>

File: mirte_modular_hardware/urdf/encoder.ros2_control.xacro (robot description, xacro)
@@ -2,5 +2,5 @@
 <robot xmlns:xacro="http://www.ros.org/wiki/xacro">
   <xacro:include filename="$(find mirte_modular_hardware)/urdf/common.xacro" />
-  <!-- NOTE; The standard slot encoders compatible with the yellow TT motors of the MIRTE Pioneer,
+  <!-- NOTE: The standard slot encoders compatible with the yellow TT motors of the MIRTE Pioneer,
              have 20 ticks per rotations -->
   <xacro:macro name="encoder_sensor"
@@ -12,8 +12,8 @@
       <hardware>
         <plugin>mirte_modular_hardware/EncoderSensor</plugin>
-        <!-- TODO PARAMS GO HERE-->
-        <!-- TODO(SuperJappie08) Check if last / already added-->
-        <!-- TODO(SuperJappie08) Ability to override topic -->
-        <!-- TODO(SuperJappie08) Ability to run inside of a namespace -->
+        <!-- TODO: PARAMS GO HERE-->
+        <!-- TODO(SuperJappie08): Check if last / already added-->
+        <!-- TODO(SuperJappie08): Ability to override topic -->
+        <!-- TODO(SuperJappie08): Ability to run inside of a namespace -->
         <param name="topic">${hardware_namespace_}/encoder/${hw_device_name}</param>
         <param name="ticks_per_rotation">${ticks_per_rotation}</param>
@@ -21,7 +21,7 @@
       </hardware>
       <joint name="${joint_name}">
-        <!-- TODO EXTRA CONFIG LIKE WRAPPING AND LIMITS -->
+        <!-- TODO: EXTRA CONFIG LIKE WRAPPING AND LIMITS -->
         <state_interface name="position" />
-        <!-- TODO(SuperJappie08) Possibly make toggleable state interface velocity? -->
+        <!-- TODO(SuperJappie08): Possibly make toggleable state interface velocity? -->
         <state_interface name="velocity" />
       </joint>

File: mirte_modular_hardware/urdf/motor.ros2_control.xacro (robot description, xacro)
@@ -7,5 +7,5 @@
     <xacro:strip_trailing_slash source="${hardware_namespace}" dest="hardware_namespace_" />
     <!-- <xacro:property name="topic_" value= scope="parent"/> -->
-    <!-- NOTE; this *highly* depends on the voltage of the motors!!!! -->
+    <!-- NOTE: this *highly* depends on the voltage of the motors!!!! -->
     <!-- For 5V power bank; 255 pwm = 90 ticks/sec -> ca 2 rot/s (4*pi) -->
     <!-- For 6V power supply; 255 pwm = 120 ticks/sec -> ca 3 rot/s (6*pi) -->
@@ -13,8 +13,8 @@
       <hardware>
         <plugin>mirte_modular_hardware/MotorActuator</plugin>
-        <!-- TODO PARAMS GO HERE-->
-        <!-- TODO(SuperJappie08) Check if last / already added-->
-        <!-- TODO(SuperJappie08) Ability to override topic -->
-        <!-- TODO(SuperJappie08) Ability to run inside of a namespace -->
+        <!-- TODO: PARAMS GO HERE-->
+        <!-- TODO(SuperJappie08): Check if last / already added-->
+        <!-- TODO(SuperJappie08): Ability to override topic -->
+        <!-- TODO(SuperJappie08): Ability to run inside of a namespace -->
         <param name="topic">${hardware_namespace_}/motor/${hw_device_name}/speed</param>
         <param name="max_motor_speed">${max_motor_speed}</param>
@@ -22,5 +22,5 @@
       <joint name="${joint_name}">
         <command_interface name="velocity" />
-        <!-- TODO EXTRA CONFIG LIKE WRAPPING AND LIMITS -->
+        <!-- TODO: Maybe make configurable like multi_motor (so based on the joint/command_interface) -->
       </joint>
     </ros2_control>

Commit message: Add old arm control

File: mirte_control/mirte_master_control/urdf/base/encoder/single_encoders.ros2_control.xacro (robot description, xacro)
@@ -10,4 +10,6 @@
       <!-- Base properties -->
       <xacro:property name="hardware_namespace_" value="${hardware_namespace or base_config.get('hardware_namespace', 'io')}" />
+      <!-- NOTE: The default if omitted is 'rw_rate="0"' which means as fast as the controller manager -->
+      <xacro:property name="rw_rate" value="${base_config.get('rw_rate', 0)}" />
       <xacro:property name="initial_message_timeout" value="${base_config.get('initial_message_timeout', 500)}" />
       <!-- Wheel specific properties -->
@@ -16,4 +18,5 @@
       <!-- wheel_name: ${wheel_name} -->
       <!-- hardware_namespace: ${hardware_namespace_} -->
+      <!-- rw_rate: ${rw_rate} Hz (0 => cm rate) -->
       <!-- initial_message_timeout: ${initial_message_timeout} ms -->
       <!-- ticks_per_rotation: ${ticks_per_rotation} -->
@@ -21,5 +24,5 @@
       <xacro:encoder_sensor hw_device_name="${wheel_name}" hardware_namespace="${hardware_namespace_}"
         joint_name="${wheel_name}_wheel_joint" initial_message_timeout="${initial_message_timeout}"
-        ticks_per_rotation="${ticks_per_rotation}"
+        ticks_per_rotation="${ticks_per_rotation}" rw_rate="${rw_rate}"
       />
       <!-- recursively call myself -->

File: mirte_control/mirte_master_control/urdf/base/motor/multi_motor.ros2_control.xacro (robot description, xacro)
@@ -29,6 +29,13 @@
     <xacro:property name="hardware_namespace_"
       value="${hardware_namespace or base_config.get('hardware_namespace', 'io')}" />
+    <!-- NOTE: The default if omitted is 'rw_rate="0"' which means as fast as the controller manager -->
+    <xacro:property name="rw_rate" value="${base_config.get('rw_rate', 0)}" />
+    <!-- xacro:eval-comments:on -->
+    <!-- hw_interface: multi_motor -->
+    <!-- hardware_namespace: ${hardware_namespace_} -->
+    <!-- rw_rate: ${rw_rate} Hz (0 => cm rate) -->
+    <!-- xacro:eval-comments:off -->
     <xacro:multi_motor_actuator hw_device_name="motorservocontroller"
-      hardware_namespace="${hardware_namespace_}">
+      hardware_namespace="${hardware_namespace_}" rw_rate="${rw_rate}">
       <joints>
         <xacro:single_multi_motor_wheel_joints wheels="${list(base_config.wheels.keys())}"

File: mirte_control/mirte_master_control/urdf/base/motor/single_motors.ros2_control.xacro (robot description, xacro)
@@ -10,4 +10,6 @@
       <!-- Base properties -->
       <xacro:property name="hardware_namespace_" value="${hardware_namespace or base_config.get('hardware_namespace', 'io')}" />
+      <!-- NOTE: The default if omitted is 'rw_rate="0"' which means as fast as the controller manager -->
+      <xacro:property name="rw_rate" value="${base_config.get('rw_rate', 0)}" />
       <!-- Wheel specific properties -->
       <xacro:property name="max_motor_speed" value="${wheel_config.max_motor_speed}"/>
@@ -15,8 +17,9 @@
       <!-- wheel_name: ${wheel_name} -->
       <!-- hardware_namespace: ${hardware_namespace_} -->
+      <!-- rw_rate: ${rw_rate} Hz (0 => cm rate) -->
       <!-- max_motor_speed: ${max_motor_speed} -->
       <!-- xacro:eval-comments:off -->
       <xacro:motor_actuator hw_device_name="${wheel_name}" hardware_namespace="${hardware_namespace_}"
-        joint_name="${wheel_name}_wheel_joint" max_motor_speed="${max_motor_speed}" />
+        joint_name="${wheel_name}_wheel_joint" max_motor_speed="${max_motor_speed}" rw_rate="${rw_rate}" />
       <!-- recursively call myself -->
       <xacro:single_motors_loop />

File: mirte_control/mirte_master_control/urdf/mirte_master_combined.urdf.xacro (robot description, xacro)
@@ -10,13 +10,17 @@
     <xacro:property name="hardware_namespace" value="$(arg hardware_namespace)" />
   </xacro:if>
-  <!-- Options: -->
-  <!-- - multi_motor -->
-  <!-- - single_motors -->
+  <!-- The options are the filenames -->
   <xacro:arg name="base_motors" default="multi_motor"/>
   <xacro:include filename="$(find mirte_master_control)/urdf/base/motor/$(arg base_motors).ros2_control.xacro"/>
   <xacro:motors base_config="${control_config.base}" />
+  <!-- The options are the filenames -->
   <xacro:arg name="base_encoders" default="single_encoders"/>
   <xacro:include filename="$(find mirte_master_control)/urdf/base/encoder/$(arg base_encoders).ros2_control.xacro"/>
   <xacro:encoders base_config="${control_config.base}" />
-  <!-- TODO: Add ARM -->
+  <!-- The options are the filenames -->
+  <xacro:arg name="hardware_interface_arm" default="old"/>
+  <xacro:if value="$(arg arm_enable)">
+    <xacro:include filename="$(find mirte_master_control)/urdf/arm/$(arg hardware_interface_arm).ros2_control.xacro"/>
+    <xacro:hardware_interface_arm arm_config="${control_config.arm if python.isinstance(control_config.get('arm'), dict) else xacro.dotify(dict())}" />
+  </xacro:if>
 </robot>

File: mirte_modular_hardware/urdf/encoder.ros2_control.xacro (robot description, xacro)
@@ -4,10 +4,11 @@
   <!-- NOTE: The standard slot encoders compatible with the yellow TT motors of the MIRTE Pioneer,
              have 20 ticks per rotations -->
+  <!-- NOTE: The default if omitted is 'rw_rate="0"' which means as fast as the controller manager -->
   <xacro:macro name="encoder_sensor"
-    params="hardware_namespace:='io' hw_device_name joint_name ticks_per_rotation:=20 initial_message_timeout:=500">
+    params="hardware_namespace:='io' hw_device_name joint_name ticks_per_rotation:=20 initial_message_timeout:=500 rw_rate:=0">
     <!-- Strip leading slash -->
     <xacro:strip_trailing_slash source="${hardware_namespace}" dest="hardware_namespace_" />
     <!-- <xacro:property name="topic_" value= scope="parent"/> -->
-    <ros2_control name="mirte_modular_hardware_encoder_${hw_device_name}" type="sensor">
+    <ros2_control name="mirte_modular_hardware_encoder_${hw_device_name}" type="sensor" rw_rate="${rw_rate}">
       <hardware>
         <plugin>mirte_modular_hardware/EncoderSensor</plugin>

File: mirte_modular_hardware/urdf/motor.ros2_control.xacro (robot description, xacro)
@@ -2,6 +2,7 @@
 <robot xmlns:xacro="http://www.ros.org/wiki/xacro">
   <xacro:include filename="$(find mirte_modular_hardware)/urdf/common.xacro" />
+  <!-- NOTE: The default if omitted is 'rw_rate="0"' which means as fast as the controller manager -->
   <xacro:macro name="motor_actuator"
-    params="hardware_namespace:='io' hw_device_name joint_name max_motor_speed:='${6.0*pi}'">
+    params="hardware_namespace:='io' hw_device_name joint_name max_motor_speed:='${6.0*pi}' rw_rate:=0">
     <!-- Strip trailing slash -->
     <xacro:strip_trailing_slash source="${hardware_namespace}" dest="hardware_namespace_" />
@@ -10,5 +11,5 @@
     <!-- For 5V power bank; 255 pwm = 90 ticks/sec -> ca 2 rot/s (4*pi) -->
     <!-- For 6V power supply; 255 pwm = 120 ticks/sec -> ca 3 rot/s (6*pi) -->
-    <ros2_control name="mirte_modular_hardware_motor_${hw_device_name}" type="actuator">
+    <ros2_control name="mirte_modular_hardware_motor_${hw_device_name}" type="actuator" rw_rate="${rw_rate}">
       <hardware>
         <plugin>mirte_modular_hardware/MotorActuator</plugin>

File: mirte_modular_hardware/urdf/multi_motor.ros2_control.xacro (robot description, xacro)
@@ -3,9 +3,10 @@
   <xacro:include filename="$(find mirte_modular_hardware)/urdf/common.xacro" />
   <xacro:include filename="$(find mirte_modular_hardware)/urdf/ros2_control.xacro" />
+  <!-- NOTE: The default if omitted is 'rw_rate="0"' which means as fast as the controller manager -->
   <xacro:macro name="multi_motor_actuator"
-    params="hardware_namespace:='io' hw_device_name **joints">
+    params="hardware_namespace:='io' hw_device_name **joints rw_rate:=0">
     <!-- Strip trailing slash -->
     <xacro:strip_trailing_slash source="${hardware_namespace}" dest="hardware_namespace_" />
-    <ros2_control name="mirte_modular_hardware_multi_motor_${hw_device_name}" type="actuator">
+    <ros2_control name="mirte_modular_hardware_multi_motor_${hw_device_name}" type="actuator" rw_rate="${rw_rate}">
       <hardware>
         <plugin>mirte_modular_hardware/MultiMotorActuator</plugin>
