Commit message: Add encoder update topic
Signed-off-by: SuperJappie08 <36795178+SuperJappie08@users.noreply.github.com>

File: mirte_control/mirte_master_control/urdf/base/encoder/single_encoders.ros2_control.xacro (robot description, xacro)
@@ -13,4 +13,5 @@
       <xacro:property name="rw_rate" value="${base_config.get('rw_rate', 0)}" />
       <xacro:property name="initial_message_timeout" value="${base_config.get('initial_message_timeout', 500)}" />
+      <xacro:property name="updates_only" value="${base_config.get('encoder_updates_only', None)}" />
       <!-- Wheel specific properties -->
       <xacro:property name="ticks_per_rotation" value="${wheel_config.ticks_per_rotation}"/>
@@ -20,9 +21,10 @@
       <!-- rw_rate: ${rw_rate} Hz (0 => cm rate) -->
       <!-- initial_message_timeout: ${initial_message_timeout} ms -->
+      <!-- updates_only: ${updates_only} -->
       <!-- ticks_per_rotation: ${ticks_per_rotation} -->
       <!-- xacro:eval-comments:off -->
       <xacro:encoder_sensor hw_device_name="${wheel_name}" hardware_namespace="${hardware_namespace_}"
         joint_name="${wheel_name}_wheel_joint" initial_message_timeout="${initial_message_timeout}"
-        ticks_per_rotation="${ticks_per_rotation}" rw_rate="${rw_rate}"
+        ticks_per_rotation="${ticks_per_rotation}" rw_rate="${rw_rate}" updates_only="${updates_only}"
       />
       <!-- recursively call myself -->

File: mirte_modular_hardware/urdf/encoder.ros2_control.xacro (robot description, xacro)
@@ -2,9 +2,10 @@
 <robot xmlns:xacro="http://www.ros.org/wiki/xacro">
   <xacro:include filename="$(find mirte_modular_hardware)/urdf/common.xacro" />
+  <xacro:include filename="$(find mirte_modular_hardware)/urdf/ros2_control.xacro" />
   <!-- NOTE: The standard slot encoders compatible with the yellow TT motors of the MIRTE Pioneer,
              have 20 ticks per rotations -->
   <!-- NOTE: The default if omitted is 'rw_rate="0"' which means as fast as the controller manager -->
   <xacro:macro name="encoder_sensor"
-    params="hardware_namespace:='io' hw_device_name joint_name ticks_per_rotation:=20 initial_message_timeout:=500 rw_rate:=0">
+    params="hardware_namespace:='io' hw_device_name joint_name ticks_per_rotation:=20 initial_message_timeout:=500 rw_rate:=0 updates_only:=${None}">
     <!-- Strip leading slash -->
     <xacro:strip_trailing_slash source="${hardware_namespace}" dest="hardware_namespace_" />
@@ -20,4 +21,5 @@
         <param name="ticks_per_rotation">${ticks_per_rotation}</param>
         <param name="initial_message_timeout_ms">${initial_message_timeout}</param>
+        <xacro:optional_param name="update" value="${updates_only}"/>
       </hardware>
       <joint name="${joint_name}">

Commit message: Add encoder message timeout after which speed 0 is assumed
Signed-off-by: SuperJappie08 <36795178+SuperJappie08@users.noreply.github.com>

File: mirte_control/mirte_master_control/urdf/base/encoder/single_encoders.ros2_control.xacro (robot description, xacro)
@@ -14,4 +14,5 @@
       <xacro:property name="initial_message_timeout" value="${base_config.get('initial_message_timeout', 500)}" />
       <xacro:property name="updates_only" value="${base_config.get('encoder_updates_only', None)}" />
+      <xacro:property name="message_timeout" value="${base_config.get('message_timeout', None)}" />
       <!-- Wheel specific properties -->
       <xacro:property name="ticks_per_rotation" value="${wheel_config.ticks_per_rotation}"/>
@@ -22,4 +23,5 @@
       <!-- initial_message_timeout: ${initial_message_timeout} ms -->
       <!-- updates_only: ${updates_only} -->
+      <!-- message_timeout: ${message_timeout} ms -->
       <!-- ticks_per_rotation: ${ticks_per_rotation} -->
       <!-- xacro:eval-comments:off -->
@@ -27,4 +29,5 @@
         joint_name="${wheel_name}_wheel_joint" initial_message_timeout="${initial_message_timeout}"
         ticks_per_rotation="${ticks_per_rotation}" rw_rate="${rw_rate}" updates_only="${updates_only}"
+        message_timeout="${message_timeout}"
       />
       <!-- recursively call myself -->

File: mirte_modular_hardware/urdf/encoder.ros2_control.xacro (robot description, xacro)
@@ -7,5 +7,5 @@
   <!-- NOTE: The default if omitted is 'rw_rate="0"' which means as fast as the controller manager -->
   <xacro:macro name="encoder_sensor"
-    params="hardware_namespace:='io' hw_device_name joint_name ticks_per_rotation:=20 initial_message_timeout:=500 rw_rate:=0 updates_only:=${None}">
+    params="hardware_namespace:='io' hw_device_name joint_name ticks_per_rotation:=20 initial_message_timeout:=500 rw_rate:=0 updates_only:=${None} message_timeout:=${None}">
     <!-- Strip leading slash -->
     <xacro:strip_trailing_slash source="${hardware_namespace}" dest="hardware_namespace_" />
@@ -22,4 +22,5 @@
         <param name="initial_message_timeout_ms">${initial_message_timeout}</param>
         <xacro:optional_param name="update" value="${updates_only}"/>
+        <xacro:optional_param name="message_timeout_ms" value="${message_timeout}"/>
       </hardware>
       <joint name="${joint_name}">

Commit message: Change velocity calculation age policy
Instead of using a set time out, just don't reuse messages.

Signed-off-by: SuperJappie08 <36795178+SuperJappie08@users.noreply.github.com>

File: mirte_control/mirte_master_control/urdf/base/encoder/single_encoders.ros2_control.xacro (robot description, xacro)
@@ -14,5 +14,4 @@
       <xacro:property name="initial_message_timeout" value="${base_config.get('initial_message_timeout', 500)}" />
       <xacro:property name="updates_only" value="${base_config.get('encoder_updates_only', None)}" />
-      <xacro:property name="message_timeout" value="${base_config.get('message_timeout', None)}" />
       <!-- Wheel specific properties -->
       <xacro:property name="ticks_per_rotation" value="${wheel_config.ticks_per_rotation}"/>
@@ -23,5 +22,4 @@
       <!-- initial_message_timeout: ${initial_message_timeout} ms -->
       <!-- updates_only: ${updates_only} -->
-      <!-- message_timeout: ${message_timeout} ms -->
       <!-- ticks_per_rotation: ${ticks_per_rotation} -->
       <!-- xacro:eval-comments:off -->
@@ -29,5 +27,4 @@
         joint_name="${wheel_name}_wheel_joint" initial_message_timeout="${initial_message_timeout}"
         ticks_per_rotation="${ticks_per_rotation}" rw_rate="${rw_rate}" updates_only="${updates_only}"
-        message_timeout="${message_timeout}"
       />
       <!-- recursively call myself -->

File: mirte_modular_hardware/urdf/encoder.ros2_control.xacro (robot description, xacro)
@@ -7,5 +7,5 @@
   <!-- NOTE: The default if omitted is 'rw_rate="0"' which means as fast as the controller manager -->
   <xacro:macro name="encoder_sensor"
-    params="hardware_namespace:='io' hw_device_name joint_name ticks_per_rotation:=20 initial_message_timeout:=500 rw_rate:=0 updates_only:=${None} message_timeout:=${None}">
+    params="hardware_namespace:='io' hw_device_name joint_name ticks_per_rotation:=20 initial_message_timeout:=500 rw_rate:=0 updates_only:=${None}">
     <!-- Strip leading slash -->
     <xacro:strip_trailing_slash source="${hardware_namespace}" dest="hardware_namespace_" />
@@ -22,5 +22,4 @@
         <param name="initial_message_timeout_ms">${initial_message_timeout}</param>
         <xacro:optional_param name="update" value="${updates_only}"/>
-        <xacro:optional_param name="message_timeout_ms" value="${message_timeout}"/>
       </hardware>
       <joint name="${joint_name}">
